Commit message: Initial backup of THOR7 ROS2 workspace

File: src/thor7v3_description/urdf/thor7v3_robot.urdf (robot description, URDF)
Before this commit: robot thor7v3, 19 links, 18 joints
Links:
- link ft_sensor_mount_link: geometry collision box size=0.022000 0.054500 0.014500; collision box size=0.026000 0.028500 0.018000
Joints:
- joint ag145_gripper_base_joint: origin xyz=0.0 0.0 0.0387 rpy=0.0 0.0 0.0 -> xyz=0.0 0.0 0.0387 rpy=0.0 0.0 -1.5707963267948966

File: src/thor7v3_description/urdf/thor7v3_robot.urdf.xacro (robot description, xacro)
@@ -25,9 +25,61 @@
          link6 +Z points outward toward the tool.
        NOTE:
-       This link is currently a kinematic mounting frame only.
-       Accurate sensor visual/collision/inertial data will be added
-       after the F/T sensor geometry/model is finalized.
+       Conservative F/T sensor collision geometry is now included
+       from the manufacturer total-assembly CAD envelope.
+       Accurate visual, inertial, and measurement-frame definitions
+       remain pending manufacturer sensor documentation.
   -->
-  <link name="ft_sensor_mount_link" />
+  <link name="ft_sensor_mount_link">
+    <!--
+      Conservative collision envelope derived from the manufacturer's
+      WF total-assembly STEP.
+      Coordinates are expressed directly in the link6 frame because
+      ft_sensor_mount_joint is identity.
+      The envelope covers:
+        - 4313S2E2-01 main F/T body
+        - 4313S2E2-02 mounting structure
+        - lateral connector / cable geometry
+      Approximately 1 mm safety margin is included.
+      IMPORTANT:
+      This is a collision envelope, not the F/T measurement frame.
+      Fx/Fy/Fz and Mx/My/Mz axes still require sensor documentation.
+    -->
+    <!-- Main F/T body + mounting structure -->
+    <collision name="ft_sensor_body_collision">
+      <origin
+        xyz="0.000000 -0.003000 0.018150"
+        rpy="0 0 0" />
+      <geometry>
+        <box size="0.085000 0.091000 0.043100" />
+      </geometry>
+    </collision>
+    <!-- Connector / cable, proximal section -->
+    <collision name="ft_sensor_cable_near_collision">
+      <origin
+        xyz="-0.058000 -0.016250 0.015500"
+        rpy="0 0 0" />
+      <geometry>
+        <box size="0.026000 0.028500 0.018000" />
+      </geometry>
+    </collision>
+    <!-- Connector / cable, middle section -->
+    <collision name="ft_sensor_cable_mid_collision">
+      <origin
+        xyz="-0.082500 0.006000 0.016350"
+        rpy="0 0 0" />
+      <geometry>
+        <box size="0.027000 0.048000 0.019700" />
+      </geometry>
+    </collision>
+    <!-- Connector / cable, distal section -->
+    <collision name="ft_sensor_cable_far_collision">
+      <origin
+        xyz="-0.105000 0.009250 0.017750"
+        rpy="0 0 0" />
+      <geometry>
+        <box size="0.022000 0.054500 0.014500" />
+      </geometry>
+    </collision>
+  </link>
   <joint name="ft_sensor_mount_joint" type="fixed">
     <parent link="link6" />
@@ -45,5 +97,5 @@
   <xacro:property
     name="gripper_mount_rpy"
-    value="0.0 0.0 0.0" />
+    value="0.0 0.0 -1.5707963267948966" />
   <xacro:dh_robotics_ag145_gripper
     prefix="ag145_"

File: src/thor7v3_moveit_config/config/thor7v3.real_dryrun.ros2_control.xacro (robot description, xacro)
@@ -1,4 +1,14 @@
 <?xml version="1.0"?>
 <robot xmlns:xacro="http://www.ros.org/wiki/xacro">
+  <!--
+    Canonical safety data. Do not duplicate numeric safe-pose values
+    in this file; edit config/thor7_safety.yaml instead.
+  -->
+  <xacro:property
+    name="thor7_safety_file"
+    value="$(find thor7v3_moveit_config)/config/thor7_safety.yaml" />
+  <xacro:property
+    name="thor7_safety"
+    value="${xacro.load_yaml(thor7_safety_file)}" />
   <xacro:macro
     name="thor7v3_real_dryrun_ros2_control"
@@ -17,16 +27,16 @@
         <param name="dry_run_command_mode">true</param>
         <!-- 启动姿态允许误差：3 degrees -->
-        <param name="startup_pose_tolerance_rad">0.0523598776</param>
+        <param name="startup_pose_tolerance_rad">${thor7_safety['startup_pose_tolerance_rad']}</param>
         <!-- 每个目标相对真实当前位置最大允许偏差：1 degree -->
-        <param name="max_command_delta_rad">0.0174532925</param>
+        <param name="max_command_delta_rad">${thor7_safety['max_command_delta_rad']}</param>
         <!-- 目标相对安全基准姿态最大允许偏差：5 degrees -->
-        <param name="max_safe_deviation_rad">0.0872664626</param>
+        <param name="max_safe_deviation_rad">${thor7_safety['max_safe_deviation_rad']}</param>
         <!-- 用户指定的安全基准姿态 -->
-        <param name="safe_j1_rad">1.876752545</param>
-        <param name="safe_j2_rad">-0.048520153</param>
-        <param name="safe_j3_rad">1.863313509</param>
-        <param name="safe_j4_rad">0.008377580</param>
-        <param name="safe_j5_rad">1.436405974</param>
-        <param name="safe_j6_rad">-0.287979327</param>
+        <param name="safe_j1_rad">${thor7_safety['safe_pose']['joint1']}</param>
+        <param name="safe_j2_rad">${thor7_safety['safe_pose']['joint2']}</param>
+        <param name="safe_j3_rad">${thor7_safety['safe_pose']['joint3']}</param>
+        <param name="safe_j4_rad">${thor7_safety['safe_pose']['joint4']}</param>
+        <param name="safe_j5_rad">${thor7_safety['safe_pose']['joint5']}</param>
+        <param name="safe_j6_rad">${thor7_safety['safe_pose']['joint6']}</param>
       </hardware>
       <joint name="joint1">

File: src/thor7v3_moveit_config/config/thor7v3.real_servoj.ros2_control.xacro (robot description, xacro)
@@ -1,4 +1,14 @@
 <?xml version="1.0"?>
 <robot xmlns:xacro="http://www.ros.org/wiki/xacro">
+  <!--
+    Canonical safety data. Do not duplicate numeric safe-pose values
+    in this file; edit config/thor7_safety.yaml instead.
+  -->
+  <xacro:property
+    name="thor7_safety_file"
+    value="$(find thor7v3_moveit_config)/config/thor7_safety.yaml" />
+  <xacro:property
+    name="thor7_safety"
+    value="${xacro.load_yaml(thor7_safety_file)}" />
   <xacro:macro
     name="thor7v3_real_servoj_ros2_control"
@@ -12,7 +22,7 @@
         <!-- Explicitly selects the only mode allowed to call servoJ(). -->
         <param name="control_mode">real_servoj</param>
-        <param name="startup_pose_tolerance_rad">0.0523598776</param>
-        <param name="max_command_delta_rad">0.0174532925</param>
-        <param name="max_safe_deviation_rad">0.0872664626</param>
+        <param name="startup_pose_tolerance_rad">${thor7_safety['startup_pose_tolerance_rad']}</param>
+        <param name="max_command_delta_rad">${thor7_safety['max_command_delta_rad']}</param>
+        <param name="max_safe_deviation_rad">${thor7_safety['max_safe_deviation_rad']}</param>
         <!-- Parameters already validated by independent real-hardware test. -->
         <param name="servoj_time_sec">0.020</param>
@@ -22,10 +32,10 @@
         <param name="servoj_command_epsilon_rad">0.000001</param>
         <param name="servoj_stop_after_stable_sec">0.5</param>
-        <param name="safe_j1_rad">1.876752545</param>
-        <param name="safe_j2_rad">-0.048520153</param>
-        <param name="safe_j3_rad">1.863313509</param>
-        <param name="safe_j4_rad">0.008377580</param>
-        <param name="safe_j5_rad">1.436405974</param>
-        <param name="safe_j6_rad">-0.287979327</param>
+        <param name="safe_j1_rad">${thor7_safety['safe_pose']['joint1']}</param>
+        <param name="safe_j2_rad">${thor7_safety['safe_pose']['joint2']}</param>
+        <param name="safe_j3_rad">${thor7_safety['safe_pose']['joint3']}</param>
+        <param name="safe_j4_rad">${thor7_safety['safe_pose']['joint4']}</param>
+        <param name="safe_j5_rad">${thor7_safety['safe_pose']['joint5']}</param>
+        <param name="safe_j6_rad">${thor7_safety['safe_pose']['joint6']}</param>
       </hardware>
       <joint name="joint1">
